Commit message: rviz display working after changing rviz config file

File: urdf/truck.urdf (robot description, URDF)
Before this commit: robot truck, 1 links, 0 joints
Links:
- removed link base_link
- added link head; visual cylinder length=0.6 radius=0.2

Commit message: truck body now visualizable with joint state publisher, but wheels not connected

File: urdf/truck.urdf (robot description, URDF)
Before this commit: robot truck, 1 links, 0 joints
Links:
- added link tail; visual box size=4 1 1
- link head: geometry visual box size=2 1 1
Joints:
- added joint link: type revolute, parent head, child tail, origin xyz=-0.5 0 0, axis 0 0 1, limit lower=-1.57 upper=1.57 effort=1000.0 velocity=10
